Commit message: updated one_leg.urdf

File: urdf/one_leg.urdf (robot description, URDF)
Before this commit: robot oneleg, 3 links, 2 joints
Links:
- removed link hip
- removed link thigh
- added link leg_link; visual cylinder length=0.14 radius=0.0127
- added link thigh_link; visual box size=0.15 0.035 0.006
- link base_link: geometry visual cylinder length=0.045 radius=0.0127
Joints:
- removed joint base_to_thigh
- removed joint thigh_to_hip
- added joint hip_to_thigh: type fixed, parent base_link, child thigh_link, origin xyz=0 0 -0.03
- added joint thigh_to_leg: type fixed, parent thigh_link, child leg_link, origin xyz=0.1246 0 -0.051 

Commit message: changed fixed joints to revolute joints

File: urdf/one_leg.urdf (robot description, URDF)
Before this commit: robot oneleg, 3 links, 2 joints
Joints:
- joint hip_to_thigh: axis (none) -> 0 1 0; limit (none) -> lower=-0.785 upper=0.785 effort=1000.0 velocity=0.5; type fixed -> revolute
- joint thigh_to_leg: axis (none) -> 0 1 0; limit (none) -> lower=-0.785 upper=0.785 effort=1000.0 velocity=0.5; origin xyz=0.1246 0 -0.051  -> xyz=0.1246 0 -0.021 ; type fixed -> revolute

Commit message: added parameterized xacro

File: urdf/one_leg.urdf (robot description, URDF)
Before this commit: robot oneleg, 3 links, 2 joints
Links:
- link base_link: mass None -> 0.03; geometry collision cylinder length=0.045 radius=0.0127; visual cylinder length=0.045 radius=0.0127
- link leg_link: mass None -> 0.03; geometry collision cylinder length=0.14 radius=0.0127; visual cylinder length=0.14 radius=0.0127
- link thigh_link: mass None -> 0.03; geometry collision box size=0.15 0.035 0.006; visual box size=0.15 0.035 0.006
