Commit message: complete 4 legs for quadruped

File: urdf/macros.xacro (robot description, xacro)
@@ -127,3 +127,15 @@
     </joint>
   </xacro:macro>
+  <!-- ############################################
+       Macro - left leg
+       ############################################ -->
+  <xacro:macro name="left_leg" params="prefix">
+    <xacro:servo suffix="${prefix}"></xacro:servo>
+    <xacro:leg prefix="${prefix}"></xacro:leg>
+    <joint name="${prefix}_hip_joint" type="fixed">
+      <parent link="servo_${prefix}_link"/>
+      <child link="${prefix}_hip_link"/>
+      <origin xyz="0 0 0"/>
+    </joint>
+  </xacro:macro>
 </robot>

Commit message: added URDF/XACRO model of the quadruped robot also added sample Python code to simulate the model in PyBullet

File: urdf/macros.xacro (robot description, xacro)
@@ -7,5 +7,5 @@
   <xacro:property name="servolen"        value="0.04" />
   <xacro:property name="servothick"      value="0.02" />
-  <xacro:property name="servo_velocity"  value="0.5" />
+  <xacro:property name="servo_velocity"  value="${60/180*pi/0.16}" />
   <xacro:property name="servo_effort"    value="1000.0" />
   <xacro:macro name="servo" params="suffix">
@@ -38,5 +38,5 @@
   <xacro:property name="thigh_mass"       value="0.03" />
   <xacro:property name="x_offset_hip_to_thigh" value="0.023" />
-  <xacro:property name="servo_velocity"  value="0.5" />
+  <xacro:property name="servo_velocity"  value="${60/180*pi/0.16}" />
   <xacro:property name="servo_effort"    value="1000.0" />
   <xacro:property name="gap_hip_to_thigh" value="0.015" />

File: urdf/quadruped.xacro (robot description, xacro)
@@ -13,4 +13,5 @@
   <xacro:property name="bodythick"       value="0.006" />
   <xacro:property name="legbaseoffset"   value="0.053" />
+  <xacro:property name="body_mass"       value="2" />
   <!-- ############################################
        Base
@@ -30,4 +31,8 @@
       <origin rpy="0 0 0" xyz="0 0 0.0"/>
     </collision>
+      <inertial>
+        <mass value="${body_mass}"/>
+        <inertia ixx="0.4" ixy="0.0" ixz="0.0" iyy="0.4" iyz="0.0" izz="0.2"/>
+      </inertial>
   </link>
   <!-- ############################################

Commit message: adding friction

File: urdf/macros.xacro (robot description, xacro)
@@ -50,4 +50,5 @@
   <xacro:property name="min_angle_leg_joint" value="-${pi/2}" />
   <xacro:property name="max_angle_leg_joint" value="${pi/2}" />
+  <xacro:property name="friction" value="0.8" />
   <!-- ############################################
        Macro - leg
@@ -113,4 +114,5 @@
         </geometry>
         <origin rpy="0 0 0" xyz="0 0 -${leg_length/2}"/>
+	<contact_coefficients mu="${friction}" />
       </collision>
       <inertial>
